File: analog_front_end.kicad_sch (KiCad schematic)
At the start: 14 parts

Commit message: design: Fix footprints library in schematic and fix drc
Parts:
- U7: footprint Package_TO_SOT_SMD:SOT-23-5 -> footprints:SOT-23-5
Changed lines of the file:
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@@
 			)
 		)
-		(property "Footprint" "Package_TO_SOT_SMD:SOT-23-5"
+		(property "Footprint" "footprints:SOT-23-5"
 			(at 86.36 111.76 0)
 			(effects
